File: cnc-grbl-lcd.kicad_pcb (KiCad board)
At the start: 2 copper layers, 47.1 x 34.3 mm, 7 parts, among them P1 ICSP-Main, P11 CTR, P12 CON, P13 TRX, P3 EXP1

Commit message: PCB tested and working
Parts:
- added C2: 0.1uF, Capacitors_SMD:C_1206, F.Cu at (197.6, 89.5)
- added C7: 20pF, Capacitors_SMD:C_1206, F.Cu at (177.9, 71.6)
- added C8: 20pF, Capacitors_SMD:C_1206, F.Cu at (177.9, 78.2)
- added IC1: ATMEGA328P-A, Housings_QFP:TQFP-32_7x7mm_Pitch0.8mm, F.Cu at (192.5, 77.1)
- added P2: ICSP, Pin_Headers:Pin_Header_Straight_2x03, F.Cu at (219.2, 90.9)
- added P4: EXP2, Pin_Headers:Pin_Header_Straight_2x05, F.Cu at (216.7, 66.3)
- added R3: 1K, Resistors_SMD:R_1206, F.Cu at (173.0, 81.3)
- added R4: 1K, Resistors_SMD:R_1206, F.Cu at (168.8, 81.3)
- added Y1: 16Mhz, Crystals:Crystal_HC49-SD_SMD, F.Cu at (182.6, 74.8)
- P3: footprint Pin_Headers:Pin_Header_Straight_2x06 -> Pin_Headers:Pin_Header_Straight_2x05
- moved P3 21.2 mm to (205.0, 66.3), turned to 0 degrees
Connections:
- P11 pad 1: RST -> (no net)
- P11 pad 3: HLD -> (no net)
- P11 pad 5: STR -> (no net)
- P3 pad 1: TX -> Beeper
- P3 pad 2: TX_FTDI -> BTN_enc
- P3 pad 3: RX -> LCDE
- P3 pad 4: RX_FTDI -> LCDRS
- P3 pad 5: reset -> LCD4
- P3 pad 6: reset-ftdi -> LCD5
- P3 pad 7: RST -> LCD6
- P3 pad 8: HLD -> LCD7
- P3 pad 9: STR -> GND
Routing:
- net +5V: track 34.9 -> 132.9 mm
- net GND: track 65.5 -> 154.4 mm, vias 1 -> 12
- net SD_CSEL: track 0.00 -> 59.5 mm
- net MISO: track 0.00 -> 56.8 mm, vias 0 -> 1
- net SCK: track 0.00 -> 51.6 mm, vias 0 -> 1
- net MOSI: track 0.00 -> 49.8 mm
- net reset-ftdi: track 29.5 -> 75.8 mm, vias 0 -> 1
- net Net-(IC1-Pad31): track 0.00 -> 26.0 mm, vias 0 -> 2
- net BTN_EN2: track 0.00 -> 24.5 mm
- net Net-(IC1-Pad30): track 0.00 -> 24.3 mm, vias 0 -> 2
- net LCDRS: track 0.00 -> 23.9 mm
- net LCD5: track 0.00 -> 23.1 mm, vias 0 -> 1
- net BTN_EN1: track 0.00 -> 21.9 mm
- net SD_DET: track 0.00 -> 20.4 mm
- net LCD7: track 0.00 -> 20.2 mm, vias 0 -> 1
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Other:
- board size 47.1 x 34.3 mm -> 60.5 x 34.3 mm
