File: cnc-grbl-lcd.sch (KiCad schematic (older format))
At the start: 7 parts, among them P1 ICSP-Main, P11 CTR, P12 CON, P13 TRX, P3 EXP1

Commit message: PCB tested and working
Parts:
- added C2: 0.1uF, Capacitors_SMD:C_1206, symbol C_Small
- added C7, C8: 20pF, Capacitors_SMD:C_1206, symbol C_Small
- added IC1: ATMEGA328P-A, Housings_QFP:TQFP-32_7x7mm_Pitch0.8mm, symbol ATMEGA328P-AU
- added P2: ICSP, Pin_Headers:Pin_Header_Straight_2x03, symbol Conn_02x03_Top_Bottom
- added P4: EXP2, Pin_Headers:Pin_Header_Straight_2x05, symbol Conn_02x05_Top_Bottom
- added R3, R4: 1K, Resistors_SMD:R_1206, symbol R
- added Y1: 16Mhz, Crystals:Crystal_HC49-SD_SMD, symbol Crystal_Small
- P1, P11, P13: symbol CONN_02X03 -> Conn_02x03_Top_Bottom
- P12: symbol CONN_02X04 -> Conn_02x04_Top_Bottom
- P3: footprint Pin_Headers:Pin_Header_Straight_2x06 -> Pin_Headers:Pin_Header_Straight_2x05; symbol CONN_02X06 -> Conn_02x05_Top_Bottom
Connections:
- net labels added: BTN_EN1, BTN_EN2, BTN_enc, Beeper, LCD4, LCD5, LCD6, LCD7, LCDE, LCDRS, MISO, MOSI, SCK, SD_CSEL, SD_DET
- net labels removed: HLD, RST, STR
- wire segments 36 -> 113
- no-connect marks 8 -> 15
Other:
- moved on the sheet: C1, C3
